File: Minerva-Hardware/PCIe-M2.kicad_sch (KiCad schematic)
At the start: 24 parts, among them J3 Bus_M.2_Socket_B, J4 Bus_M.2_Socket_M, J7 JAE_SIM_Card_SF72S006, M6 M.2 Solder Nut, M7 M.2 Screw, U2 ASEK-32.768KHZ-L-R-T, U8 AP3441SHE-7B

Commit message: working on pcb more
Connections:
- no-connect marks 48 -> 52
Changed lines of the file:
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@@
 	)
 	(junction
+		(at 113.03 167.64)
+		(diameter 0)
+		(color 0 0 0 0)
+	)
+	(junction
 		(at 109.22 175.26)
 		(diameter 0)
@@
 	)
 	(no_connect
-		(at 96.52 116.84)
+		(at 255.27 96.52)
 	)
 	(no_connect
@@
 	)
 	(no_connect
-		(at 96.52 114.3)
+		(at 255.27 73.66)
 	)
 	(no_connect
-		(at 255.27 73.66)
+		(at 255.27 25.4)
 	)
 	(no_connect
@@
 	)
 	(no_connect
+		(at 255.27 88.9)
+	)
+	(no_connect
 		(at 255.27 71.12)
 	)
@@
 	)
 	(no_connect
+		(at 255.27 27.94)
+	)
+	(no_connect
 		(at 255.27 106.68)
 	)
@@
 	)
 	(no_connect
-		(at 96.52 119.38)
+		(at 204.47 91.44)
 	)
 	(no_connect
@@
 	)
 	(no_connect
+		(at 255.27 33.02)
+	)
+	(no_connect
 		(at 45.72 62.23)
 	)
@@
 	)
 	(no_connect
+		(at 255.27 30.48)
+	)
+	(no_connect
 		(at 255.27 104.14)
 	)
@@
 	(wire
 		(pts
-			(xy 189.23 48.26) (xy 204.47 48.26)
-		)
-		(stroke
-			(width 0)
-			(type default)
-		)
-	)
-	(wire
-		(pts
-			(xy 175.26 97.79) (xy 175.26 96.52)
+			(xy 200.66 48.26) (xy 204.47 48.26)
 		)
 		(stroke
@@
 	(wire
 		(pts
-			(xy 176.53 93.98) (xy 175.26 93.98)
+			(xy 175.26 93.98) (xy 180.34 93.98)
 		)
 		(stroke
@@
 	(wire
 		(pts
-			(xy 109.22 167.64) (xy 119.38 167.64)
+			(xy 109.22 167.64) (xy 113.03 167.64)
 		)
 		(stroke
@@
 	(wire
 		(pts
-			(xy 142.24 167.64) (xy 152.4 167.64)
-		)
-		(stroke
-			(width 0)
-			(type default)
-		)
-	)
-	(wire
-		(pts
 			(xy 88.9 165.1) (xy 88.9 170.18)
 		)
@@
 	(wire
 		(pts
-			(xy 152.4 167.64) (xy 162.56 167.64)
-		)
-		(stroke
-			(width 0)
-			(type default)
-		)
-	)
-	(wire
-		(pts
 			(xy 59.69 162.56) (xy 64.77 162.56)
 		)
@@
 	(wire
 		(pts
-			(xy 176.53 95.25) (xy 176.53 93.98)
-		)
-		(stroke
-			(width 0)
-			(type default)
-		)
-	)
-	(wire
-		(pts
 			(xy 101.6 92.71) (xy 101.6 88.9)
 		)
@@
 	(wire
 		(pts
-			(xy 143.51 110.49) (xy 96.52 110.49)
+			(xy 113.03 167.64) (xy 162.56 167.64)
 		)
 		(stroke
@@
 	(wire
 		(pts
-			(xy 96.52 92.71) (xy 101.6 92.71)
+			(xy 143.51 110.49) (xy 96.52 110.49)
 		)
 		(stroke
@@
 	(wire
 		(pts
-			(xy 74.93 34.29) (xy 77.47 34.29)
+			(xy 96.52 92.71) (xy 101.6 92.71)
 		)
 		(stroke
@@
 	(wire
 		(pts
-			(xy 46.99 167.64) (xy 55.88 167.64)
+			(xy 74.93 34.29) (xy 77.47 34.29)
 		)
 		(stroke
@@
 	(wire
 		(pts
-			(xy 177.8 92.71) (xy 177.8 91.44)
+			(xy 46.99 167.64) (xy 55.88 167.64)
 		)
 		(stroke
@@
 	(wire
 		(pts
-			(xy 132.08 167.64) (xy 142.24 167.64)
-		)
-		(stroke
-			(width 0)
-			(type default)
-		)
-	)
-	(wire
-		(pts
 			(xy 101.6 74.93) (xy 101.6 81.28)
 		)
@@
 	(wire
 		(pts
-			(xy 189.23 58.42) (xy 204.47 58.42)
+			(xy 200.66 58.42) (xy 204.47 58.42)
 		)
 		(stroke
@@
 	(wire
 		(pts
-			(xy 175.26 83.82) (xy 193.04 83.82)
+			(xy 113.03 162.56) (xy 113.03 167.64)
 		)
 		(stroke
@@
 	(wire
 		(pts
-			(xy 119.38 167.64) (xy 132.08 167.64)
+			(xy 175.26 83.82) (xy 193.04 83.82)
 		)
 		(stroke
@@
 	(wire
 		(pts
-			(xy 189.23 53.34) (xy 204.47 53.34)
+			(xy 200.66 53.34) (xy 204.47 53.34)
 		)
 		(stroke
@@
 	(wire
 		(pts
-			(xy 180.34 97.79) (xy 175.26 97.79)
+			(xy 180.34 96.52) (xy 175.26 96.52)
 		)
 		(stroke
@@
 	(wire
 		(pts
-			(xy 177.8 91.44) (xy 175.26 91.44)
+			(xy 175.26 91.44) (xy 180.34 91.44)
 		)
 		(stroke
@@
 	(wire
 		(pts
-			(xy 143.51 130.81) (xy 129.54 130.81)
+			(xy 255.27 78.74) (xy 265.43 78.74)
 		)
 		(stroke
@@
 	(wire
 		(pts
-			(xy 176.53 95.25) (xy 180.34 95.25)
+			(xy 143.51 130.81) (xy 129.54 130.81)
 		)
 		(stroke
@@
 	(wire
 		(pts
-			(xy 179.07 111.76) (xy 179.07 115.57)
+			(xy 179.07 111.76) (xy 179.07 113.03)
 		)
 		(stroke
@@
 	(wire
 		(pts
-			(xy 189.23 60.96) (xy 204.47 60.96)
+			(xy 200.66 60.96) (xy 204.47 60.96)
 		)
 		(stroke
@@
 	(wire
 		(pts
-			(xy 189.23 50.8) (xy 204.47 50.8)
+			(xy 200.66 50.8) (xy 204.47 50.8)
 		)
 		(stroke
@@
 	(wire
 		(pts
-			(xy 189.23 45.72) (xy 204.47 45.72)
+			(xy 200.66 45.72) (xy 204.47 45.72)
 		)
 		(stroke
@@
 	(wire
 		(pts
-			(xy 177.8 92.71) (xy 180.34 92.71)
-		)
-		(stroke
-			(width 0)
-			(type default)
-		)
-	)
-	(wire
-		(pts
 			(xy 40.64 39.37) (xy 45.72 39.37)
 		)
@@
 	)
 	(label "M2_3v3"
-		(at 154.94 167.64 0)
+		(at 113.03 162.56 180)
 		(effects
 			(font
 				(size 1.27 1.27)
 			)
-			(justify left bottom)
+			(justify right bottom)
 		)
 	)
@@
 	)
 	(label "SIM_VCC"
-		(at 180.34 97.79 0)
+		(at 180.34 96.52 0)
 		(effects
 			(font
@@
 	)
 	(label "SIM_CLK"
-		(at 180.34 92.71 0)
+		(at 180.34 91.44 0)
 		(effects
 			(font
@@
 	)
 	(label "SIM_RST"
-		(at 180.34 95.25 0)
+		(at 180.34 93.98 0)
 		(effects
 			(font
@@
 	(hierarchical_label "MODEM_USBTX_N"
 		(shape bidirectional)
-		(at 189.23 48.26 180)
+		(at 200.66 48.26 180)
 		(effects
 			(font
@@
 	(hierarchical_label "MODEM_USBD_P"
 		(shape bidirectional)
-		(at 189.23 58.42 180)
+		(at 200.66 58.42 180)
 		(effects
 			(font
@@
 	(hierarchical_label "MODEM_USBD_N"
 		(shape bidirectional)
-		(at 189.23 60.96 180)
+		(at 200.66 60.96 180)
 		(effects
 			(font
@@
 	(hierarchical_label "MODEM_USBRX_N"
 		(shape bidirectional)
-		(at 189.23 53.34 180)
+		(at 200.66 53.34 180)
 		(effects
 			(font
@@
 	)
 	(hierarchical_label "PERST"
-		(shape output)
+		(shape bidirectional)
 		(at 200.66 25.4 180)
 		(effects
@@
 	(hierarchical_label "MODEM_USBRX_P"
 		(shape bidirectional)
-		(at 189.23 50.8 180)
+		(at 200.66 50.8 180)
 		(effects
 			(font
@@
 	(hierarchical_label "MODEM_USBTX_P"
 		(shape bidirectional)
-		(at 189.23 45.72 180)
+		(at 200.66 45.72 180)
 		(effects
 			(font
@@
 	(symbol
 		(lib_id "power:GND")
-		(at 179.07 115.57 0)
+		(at 179.07 113.03 0)
 		(unit 1)
 		(body_style 1)
@@
 		(fields_autoplaced yes)
 		(property "Reference" "#PWR027"
-			(at 179.07 121.92 0)
+			(at 179.07 119.38 0)
 			(hide yes)
 			(show_name no)
@@
 		)
 		(property "Value" "GND"
-			(at 179.07 120.65 0)
+			(at 179.07 118.11 0)
 			(show_name no)
 			(do_not_autoplace no)
@@
 		)
 		(property "Footprint" ""
-			(at 179.07 115.57 0)
+			(at 179.07 113.03 0)
 			(hide yes)
 			(show_name no)
@@
 		)
 		(property "Datasheet" ""
-			(at 179.07 115.57 0)
+			(at 179.07 113.03 0)
 			(hide yes)
 			(show_name no)
@@
 		)
 		(property "Description" "Power symbol creates a global label with name \"GND\" , ground"
-			(at 179.07 115.57 0)
+			(at 179.07 113.03 0)
 			(hide yes)
 			(show_name no)
@@
 		(in_pos_files yes)
 		(dnp no)
-		(fields_autoplaced yes)
 		(property "Reference" "#PWR026"
 			(at 181.61 88.9 0)
@@
 		)
 		(property "Value" "GND"
-			(at 179.07 88.8999 90)
+			(at 178.308 87.376 90)
 			(show_name no)
 			(do_not_autoplace no)
