File: Minerva-Hardware/PCIe-M2.kicad_sch (KiCad schematic)
At the start: 24 parts, among them J3 Bus_M.2_Socket_B, J4 Bus_M.2_Socket_M, J7 JAE_SIM_Card_SF72S006, M6 M.2 Solder Nut, M7 M.2 Screw, U2 ASEK-32.768KHZ-L-R-T, U8 AP3441SHE-7B

Commit message: Capture pre-existing Minerva hardware and Torchform work
Hardware schematics and power architecture
- Update carrier, CM5 GPIO, high-speed, PCIe/M.2, face-board, and root schematic hierarchy.
- Add USB-C/DisplayPort dock path, PD controller support, display bridge, audio amplifier, battery charging, boost conversion, fuel gauge, RTC backup, and MCU interconnect changes.
- Add the relocated power/USB schematic and associated local symbols, footprints, and 3D models.

PCB and design assets
- Update the carrier PCB and project configuration.
- Add CM5, connector, power, battery, PD, and board-specific footprint libraries.
- Add the USB-C receptacle STEP model and supporting KiCad assets.
- Apply the surfaced carrier-board geometry cleanup and add the J23 shell-peg DRC rule.

Verification and reference material
- Add CM5 and component datasheets, extracted reference text, current netlist, DRC output, and hardware verification documentation.
- Update CONTEXT.md and workspace metadata with the current project state.

Torchform companion projects
- Add the standalone Qt/QML gamepad prototype.
- Add the Torchform QML GUI shell with screen, panel, radial-menu, keyboard, status, and startup components.
- Add the companion Rust input daemon prototype and configuration.

Project notes
- Add repository guidance and Minerva design/editor notes, including the power-usage note.
Parts:
- added R84: 100kΩ, Resistor_SMD:R_0402_1005Metric, symbol Device:R
- C12, C13: footprint (none) -> Capacitor_SMD:C_0402_1005Metric
- J3: symbol Connector:Bus_M.2_Socket_B -> Minerva_Dock:Bus_M.2_Socket_B
- L1: footprint CM5IO:L_Bourns_SRP5030CC -> Inductor_SMD:L_Bourns_SRP5030T
- M6: footprint (none) -> MountingHole:MountingHole_2.2mm_M2_DIN965_Pad
- M7: footprint (none) -> MountingHole:MountingHole_2.2mm_M2
Connections:
- net M2_3v3: now also R84.1
- net M2_FCPO: now reaches J3.6 (~{FULL_CARD_POWER_OFF})
- net M2_FCPO: now also R84.2
- no-connect marks 52 -> 54

Commit message: hardware: snapshot carrier and face-board integration
Hardware schematics and power:
- complete the BQ25798 charger, TPS61088 5 V boost, MAX17048 gauge, battery controls, and cross-sheet power hierarchy
- add the SN65DSI86 display bridge, HD3SS460 mux, TPS65987D PD controller, USB-C protection, M.2 support, and corrected named-interface wiring
- move the Core2350B0 onto the face-board interconnect, route controls through J25/J2, and make Select directly assert nRPIBOOT
- remove the obsolete J6/J8 expansion headers and move J23 USB-C to the carrier top-left with its VBUS switch and charger support cluster

PCB, footprints, and mechanical assets:
- establish the six-layer controlled-impedance carrier stack, net classes, HDI rules, ground/power planes, keepouts, and placed carrier floorplan
- add the routed two-layer Minerva-Face board with eleven controls, four M2.5 holes, interconnects, fiducials, and a 3.5-inch display datum
- add corrected project-local footprints and STEP models for Core2350B0, USB-C, bridge/PD/power ICs, PicoBlade connectors, M.2 hardware, and critical mechanical envelopes
- correct BAT54 pin mapping, TPS61088 thermal-via numbering, J23 shell geometry, and board-edge lug rules

Verification and reference material:
- add sourcing evidence, ERC/DRC artifacts, STEP assemblies, face render, mechanical coordinates, controlled-impedance notes, and strict connectivity checklists
- document the dock architecture and current board-to-board pin contract
- remove transient root-level DRC and netlist dumps

Torchform and workstation integration:
- fix four-column home navigation and add controller focus/adjustment for quick-settings volume and brightness sliders
- configure Kitty as the terminal backend and add the Minerva SSH workspace folder

Known work-in-progress at this snapshot:
- carrier schematic/PCB parity is clean, but routing remains incomplete at 499 unconnected items with 53 differential-pair tuning violations
- the face board is DRC-clean and f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
Parts:
- C10, C20: MPN (none) -> EMK105B7104KV-F; Manufacturer (none) -> Taiyo Yuden
- C11: MPN (none) -> GRM155R71H472KA01D; Manufacturer (none) -> Murata
- C12, C13: value C -> 100nF; MPN (none) -> EMK105B7104KV-F; Manufacturer (none) -> Taiyo Yuden
- C14, C15, C16, C17, C4, C6: MPN (none) -> CL21A106KPFNNNE; Manufacturer (none) -> Samsung Electro-Mechanics
- D5: MPN (none) -> SML-A12M8TT86; Manufacturer (none) -> ROHM
- J3: MPN (none) -> 1-2199230-3; Manufacturer (none) -> TE Connectivity
- J4: MPN (none) -> 1-2199230-6; Manufacturer (none) -> TE Connectivity
- J7: MPN (none) -> SF72S006VBDR2500; Manufacturer (none) -> JAE
- L1: MPN (none) -> SRP5030CC-2R2M; Manufacturer (none) -> Bourns
- M6: value M.2 Solder Nut -> SMTSO-M2-4ET M2 standoff; footprint MountingHole:MountingHole_2.2mm_M2_DIN965_Pad -> Minerva:SMTSO-M2-4ET; MPN (none) -> SMTSO-M2-4ET; Manufacturer (none) -> PennEngineering (PEM); Procurement Note (none) -> M2 x 0.4 ReelFast surface-mount standoff, 4 mm height, 6.2 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
- M7: value M.2 Screw -> M2x3 DIN 7985H screw; footprint MountingHole:MountingHole_2.2mm_M2 -> (none); MPN (none) -> M2X3-DIN7985H-A2; Manufacturer (none) -> ISO/DIN commodity; Procurement Note (none) -> M2 x 3 mm, 0.4 mm pitch, A2 stainless Phillips pan-head scr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
- R14, R84: MPN (none) -> RC0402FR-07100KL; Manufacturer (none) -> Yageo
- R15: MPN (none) -> RC0402FR-0710KL; Manufacturer (none) -> Yageo
- R16: MPN (none) -> RT0402FRE072K2L; Manufacturer (none) -> Yageo
- R3: MPN (none) -> RK73H1ETTP1001F; Manufacturer (none) -> KOA Speer
- U2: MPN (none) -> ASEK-32.768KHZ-L-R-T; Manufacturer (none) -> Abracon
- U8: MPN (none) -> AP3441SHE-7B; Manufacturer (none) -> Diodes Incorporated
