File: Minerva-Hardware/Minerva-Carrier.kicad_sch (KiCad schematic)
At the start: 33 parts, among them J11 USB_C_Receptacle_USB2.0, U1 BQ25798

Commit message: wip shit
Other:
- company: Copyright © 2024 Raspberry Pi Ltd. -> Zack Dell
- title: Compute Module 5 IO Board - Top Level -> Minerva Carrier Board
- moved on the sheet: D4, H2, H3, R2
Changed lines of the file:
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@@
 	(paper "A4")
 	(title_block
-		(title "Compute Module 5 IO Board - Top Level")
+		(title "Minerva Carrier Board")
 		(rev "1")
-		(company "Copyright © 2024 Raspberry Pi Ltd.")
-		(comment 1 "www.raspberrypi.com")
+		(company "Zack Dell")
+		(comment 1 "zackdell.com")
 	)
 	(text "Connectors\n-------\n40way RPI\nJumpers\nFan\nBattery"
@@
 	(wire
 		(pts
-			(xy 147.32 168.91) (xy 148.59 168.91)
+			(xy 97.79 177.8) (xy 99.06 177.8)
 		)
 		(stroke
@@
 	(wire
 		(pts
-			(xy 157.48 168.91) (xy 157.48 170.18)
+			(xy 107.95 177.8) (xy 107.95 179.07)
 		)
 		(stroke
@@
 	(wire
 		(pts
-			(xy 156.21 168.91) (xy 157.48 168.91)
+			(xy 106.68 177.8) (xy 107.95 177.8)
 		)
 		(stroke
@@
 	(wire
 		(pts
-			(xy 140.97 168.91) (xy 142.24 168.91)
+			(xy 91.44 177.8) (xy 92.71 177.8)
 		)
 		(stroke
@@
 	)
 	(label "CRG_IND_SIG"
-		(at 140.97 168.91 180)
+		(at 91.44 177.8 180)
 		(effects
 			(font
@@
 	(symbol
 		(lib_id "Mechanical:MountingHole")
-		(at 22.86 175.895 0)
+		(at 248.92 113.03 0)
 		(unit 1)
 		(body_style 1)
@@
 		(dnp yes)
 		(property "Reference" "H3"
-			(at 25.4 174.752 0)
+			(at 251.46 111.887 0)
 			(show_name no)
 			(do_not_autoplace no)
@@
 		)
 		(property "Value" "MountingHole"
-			(at 25.4 177.038 0)
+			(at 251.46 114.173 0)
 			(show_name no)
 			(do_not_autoplace no)
@@
 		)
 		(property "Footprint" "CM5IO:MountingHole_2.7mm_M2.5_DIN965"
-			(at 22.86 175.895 0)
+			(at 248.92 113.03 0)
 			(hide yes)
 			(show_name no)
@@
 		)
 		(property "Datasheet" ""
-			(at 22.86 175.895 0)
+			(at 248.92 113.03 0)
 			(hide yes)
 			(show_name no)
@@
 		)
 		(property "Description" "Mounting Hole without connection"
-			(at 22.86 175.895 0)
+			(at 248.92 113.03 0)
 			(hide yes)
 			(show_name no)
@@
 		)
 		(property "Field4" "nf"
-			(at 22.86 175.895 0)
+			(at 248.92 113.03 0)
 			(hide yes)
 			(show_name no)
@@
 		)
 		(property "Field5" "nf"
-			(at 22.86 175.895 0)
+			(at 248.92 113.03 0)
 			(hide yes)
 			(show_name no)
@@
 		)
 		(property "Field6" "nf"
-			(at 22.86 175.895 0)
+			(at 248.92 113.03 0)
 			(hide yes)
 			(show_name no)
@@
 		)
 		(property "Field7" "nf"
-			(at 22.86 175.895 0)
+			(at 248.92 113.03 0)
 			(hide yes)
 			(show_name no)
@@
 		)
 		(property "Part Description" "M2.5 mounting hole"
-			(at 22.86 175.895 0)
+			(at 248.92 113.03 0)
 			(hide yes)
 			(show_name no)
@@
 	(symbol
 		(lib_id "Mechanical:MountingHole")
-		(at 22.86 170.815 0)
+		(at 248.92 107.95 0)
 		(unit 1)
 		(body_style 1)
@@
 		(dnp yes)
 		(property "Reference" "H2"
-			(at 25.4 169.672 0)
+			(at 251.46 106.807 0)
 			(show_name no)
 			(do_not_autoplace no)
@@
 		)
 		(property "Value" "MountingHole"
-			(at 25.4 171.958 0)
+			(at 251.46 109.093 0)
 			(show_name no)
 			(do_not_autoplace no)
@@
 		)
 		(property "Footprint" "CM5IO:MountingHole_2.7mm_M2.5_DIN965"
-			(at 22.86 170.815 0)
+			(at 248.92 107.95 0)
 			(hide yes)
 			(show_name no)
@@
 		)
 		(property "Datasheet" ""
-			(at 22.86 170.815 0)
+			(at 248.92 107.95 0)
 			(hide yes)
 			(show_name no)
@@
 		)
 		(property "Description" "Mounting Hole without connection"
-			(at 22.86 170.815 0)
+			(at 248.92 107.95 0)
 			(hide yes)
 			(show_name no)
@@
 		)
 		(property "Field4" "nf"
-			(at 22.86 170.815 0)
+			(at 248.92 107.95 0)
 			(hide yes)
 			(show_name no)
@@
 		)
 		(property "Field5" "nf"
-			(at 22.86 170.815 0)
+			(at 248.92 107.95 0)
 			(hide yes)
 			(show_name no)
@@
 		)
 		(property "Field6" "nf"
-			(at 22.86 170.815 0)
+			(at 248.92 107.95 0)
 			(hide yes)
 			(show_name no)
@@
 		)
 		(property "Field7" "nf"
-			(at 22.86 170.815 0)
+			(at 248.92 107.95 0)
 			(hide yes)
 			(show_name no)
@@
 		)
 		(property "Part Description" "M2.5 mounting hole"
-			(at 22.86 170.815 0)
+			(at 248.92 107.95 0)
 			(hide yes)
 			(show_name no)
@@
 	(symbol
 		(lib_id "Device:R_Small_US")
-		(at 144.78 168.91 90)
+		(at 95.25 177.8 90)
 		(unit 1)
 		(body_style 1)
@@
 		(fields_autoplaced yes)
 		(property "Reference" "R2"
-			(at 144.78 162.56 90)
+			(at 95.25 171.45 90)
 			(show_name no)
 			(do_not_autoplace no)
@@
 		)
 		(property "Value" "10k"
-			(at 144.78 165.1 90)
+			(at 95.25 173.99 90)
 			(show_name no)
 			(do_not_autoplace no)
@@
 		)
 		(property "Footprint" "Resistor_SMD:R_0201_0603Metric"
-			(at 144.78 168.91 0)
+			(at 95.25 177.8 0)
 			(hide yes)
 			(show_name no)
@@
 		)
 		(property "Datasheet" ""
-			(at 144.78 168.91 0)
+			(at 95.25 177.8 0)
 			(hide yes)
 			(show_name no)
@@
 		)
 		(property "Description" "Resistor, small US symbol"
-			(at 144.78 168.91 0)
+			(at 95.25 177.8 0)
 			(hide yes)
 			(show_name no)
@@
 	(symbol
 		(lib_id "Device:LED")
-		(at 152.4 168.91 180)
+		(at 102.87 177.8 180)
 		(unit 1)
 		(body_style 1)
@@
 		(fields_autoplaced yes)
 		(property "Reference" "D4"
-			(at 153.9875 161.29 0)
+			(at 104.4575 170.18 0)
 			(show_name no)
 			(do_not_autoplace no)
@@
 		)
 		(property "Value" "LED"
-			(at 153.9875 163.83 0)
+			(at 104.4575 172.72 0)
 			(show_name no)
 			(do_not_autoplace no)
@@
 		)
 		(property "Footprint" "LED_SMD:LED_0201_0603Metric"
-			(at 152.4 168.91 0)
+			(at 102.87 177.8 0)
 			(hide yes)
 			(show_name no)
@@
 		)
 		(property "Datasheet" ""
-			(at 152.4 168.91 0)
+			(at 102.87 177.8 0)
 			(hide yes)
 			(show_name no)
@@
 		)
 		(property "Description" "Light emitting diode"
-			(at 152.4 168.91 0)
+			(at 102.87 177.8 0)
 			(hide yes)
 			(show_name no)
@@
 		)
 		(property "Sim.Pins" "1=K 2=A"
-			(at 152.4 168.91 0)
+			(at 102.87 177.8 0)
 			(hide yes)
 			(show_name no)
@@
 	(symbol
 		(lib_id "power:GND")
-		(at 157.48 170.18 0)
+		(at 107.95 179.07 0)
 		(unit 1)
 		(body_style 1)
@@
 		(fields_autoplaced yes)
 		(property "Reference" "#PWR04"
-			(at 157.48 176.53 0)
+			(at 107.95 185.42 0)
 			(hide yes)
 			(show_name no)
@@
 		)
 		(property "Value" "GND"
-			(at 157.48 175.26 0)
+			(at 107.95 184.15 0)
 			(show_name no)
 			(do_not_autoplace no)
@@
 		)
 		(property "Footprint" ""
-			(at 157.48 170.18 0)
+			(at 107.95 179.07 0)
 			(hide yes)
 			(show_name no)
@@
 		)
 		(property "Datasheet" ""
-			(at 157.48 170.18 0)
+			(at 107.95 179.07 0)
 			(hide yes)
 			(show_name no)
@@
 		)
 		(property "Description" "Power symbol creates a global label with name \"GND\" , ground"
-			(at 157.48 170.18 0)
+			(at 107.95 179.07 0)
 			(hide yes)
 			(show_name no)

Commit message: need to improve diff pair routing
Other:
- company: Zack Dell -> (none)
Changed lines of the file:
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@@
 		(title "Minerva Carrier Board")
 		(rev "1")
-		(company "Zack Dell")
-		(comment 1 "zackdell.com")
 	)
 	(text "Connectors\n-------\n40way RPI\nJumpers\nFan\nBattery"
