File: Minerva-Hardware/CM5_GPIO.kicad_sch (KiCad schematic)
At the start: 14 parts, among them J14 JST_SHBM04B-SRSS-TB, J2 Conn_02x07_Odd_Even, J8 THD-20-R, SW1 Right angle Tact button

Commit message: Capture pre-existing Minerva hardware and Torchform work
Hardware schematics and power architecture
- Update carrier, CM5 GPIO, high-speed, PCIe/M.2, face-board, and root schematic hierarchy.
- Add USB-C/DisplayPort dock path, PD controller support, display bridge, audio amplifier, battery charging, boost conversion, fuel gauge, RTC backup, and MCU interconnect changes.
- Add the relocated power/USB schematic and associated local symbols, footprints, and 3D models.

PCB and design assets
- Update the carrier PCB and project configuration.
- Add CM5, connector, power, battery, PD, and board-specific footprint libraries.
- Add the USB-C receptacle STEP model and supporting KiCad assets.
- Apply the surfaced carrier-board geometry cleanup and add the J23 shell-peg DRC rule.

Verification and reference material
- Add CM5 and component datasheets, extracted reference text, current netlist, DRC output, and hardware verification documentation.
- Update CONTEXT.md and workspace metadata with the current project state.

Torchform companion projects
- Add the standalone Qt/QML gamepad prototype.
- Add the Torchform QML GUI shell with screen, panel, radial-menu, keyboard, status, and startup components.
- Add the companion Rust input daemon prototype and configuration.

Project notes
- Add repository guidance and Minerva design/editor notes, including the power-usage note.
Parts:
- removed J2: Conn_02x07_Odd_Even, Connector_PinHeader_2.54mm:PinHeader_2x07_P2.54mm_Vertical, symbol Connector_Generic:Conn_02x07_Odd_Even
- added BT3: ML1220, Battery:BatteryHolder_Keystone_3000_1x12mm, symbol Device:Battery_Cell
- added C100, C101, C99: 1uF, Capacitor_SMD:C_0402_1005Metric, symbol Device:C
- added C95, C97: 100nF, Capacitor_SMD:C_0402_1005Metric, symbol Device:C
- added C96, C98: 10uF, Capacitor_SMD:C_0603_1608Metric, symbol Device:C
- added D6, D7: BAT54, Minerva:D_SOT-23_BAT54_AK, symbol Device:D_Schottky
- added J20, J21: SPK_1.25mm_4P, Connector_Molex:Molex_PicoBlade_53398-0471_1x04-1MP_P1.25mm_Vertical, symbol Connector_Generic:Conn_01x04
- added J22: AUX_IN_3.5mm, Connector_JST:JST_SH_BM03B-SRSS-TB_1x03-1MP_P1.00mm_Vertical, symbol Connector_Generic:Conn_01x03
- added J25: FACEPLATE 14P, Connector_Molex:Molex_PicoBlade_53047-1410_1x14_P1.25mm_Vertical, symbol Connector_Generic:Conn_01x14
- added R71, R72: 100K, Resistor_SMD:R_0402_1005Metric, symbol Device:R
- added R75: 1kΩ, Resistor_SMD:R_0402_1005Metric, symbol Device:R
- added R85, R86: 2.2kΩ, Resistor_SMD:R_0402_1005Metric, symbol Device:R
- added U29: PAM8406DR, Package_SO:SOIC-16_3.9x9.9mm_P1.27mm, symbol Minerva_Dock:PAM8406
Connections:
- net GPIO2 is gone; now on net SDA_I2C: J8.3 (Pin_3), Module1.58 (GPIO2)
- net GPIO3 is gone; now on net SCL_I2C: J8.5 (Pin_5), Module1.56 (GPIO3)
- net +3.3v: now also R75.1, R85.1, R86.1
- net +5v: now also C95.1, C96.1, C97.1, C98.1, J25.1 (Pin_1), R71.1, R72.1, U29.13 (PVDDR), U29.4 (PVDDL), U29.6 (VDD), U29.9 (MODE)
- net GND: now also BT3.2 (-), C101.2, C95.2, C96.2, C97.2, C98.2, J22.3 (Pin_3), J25.14 (Pin_14), J25.2 (Pin_2), U29.11 (GND), U29.15 (PGNDR), U29.2 (PGNDL)
- net PWR_BUT: now also D6.1 (K), J25.10 (Pin_10)
- net SCL_I2C: now also J25.7 (Pin_7), R86.2
- net SDA_I2C: now also J25.6 (Pin_6), R85.2
- net VBAT: now also BT3.1 (+), D7.1 (K)
- net nRPIBOOT: now also J25.11 (Pin_11)
- net GPIO26 renamed DSI86_EN
- net PMIC_ENABLE: no longer names the net of Module1.99 (PMIC_ENABLE)
- new net AMP_nMUTE: J25.12 (Pin_12), R71.2, U29.5 (~{MUTE})
- new net AMP_nSD: J25.13 (Pin_13), R72.2, U29.12 (~{SHDN})
- new net AUX_L: C99.1, J22.1 (Pin_1)
- new net AUX_R: C100.1, J22.2 (Pin_2)
- new net BQ_SCL: J25.9 (Pin_9)
- new net BQ_SDA: J25.8 (Pin_8)
- new net PAM_INL: C99.2, U29.7 (INL)
- new net PAM_INR: C100.2, U29.10 (INR)
- new net PAM_VREF: C101.1, U29.8 (VREF)
- new net PD_I2C_IRQ: J25.5 (Pin_5)
- new net PD_I2C_SCL: J25.4 (Pin_4)
- new net PD_I2C_SDA: J25.3 (Pin_3)
- new net QON: D6.2 (A)
- new net SPK_L_N: J20.3 (Pin_3), J20.4 (Pin_4), U29.3 (-OUT_L)
- new net SPK_L_P: J20.1 (Pin_1), J20.2 (Pin_2), U29.1 (+OUT_L)
- new net SPK_R_N: J21.3 (Pin_3), J21.4 (Pin_4), U29.14 (-OUT_R)
- new net SPK_R_P: J21.1 (Pin_1), J21.2 (Pin_2), U29.16 (+OUT_R)
- new net VBAT_CHG: D7.2 (A), R75.2
- no-connect marks 27 -> 26
Other:
- note added: "AUDIO + DOCK MCU U29 PAM8406: stereo class-D amp fed from the upper display's 3.5mm HDMI-audio jack via J22 pigtail (tip=L ring=R sleeve=GND). MODE=+5v -> Class-D. 1uF input caps. ~MUTE/~SHDN pulled to +5v via 100K; RP2350B may pull low OPEN-DRAIN ONLY (5V net). BTL outputs: no caps, no ground on OUT-. J20/J21 pins 1-2=+, 3-4=-. NOTE: volume is the HDMI/display path volume; keep aux wiring away f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"
- note added: "Faceplate interconnect - RP2350B (Core2350B) lives on the face board"
- note added: "RTC backup: BT3 = ML1220 RECHARGEABLE only (trickled from 3.3v via R75+D7 ~= 3.0 V). If fitting a CR1220 primary cell instead: DNP R75 and D7. D6: power button also pulls BQ25798 ~QON low - hold >15 s with adapter absent = ship mode exit/entry."
- note removed: "Force RPIBOOT = Jumper Pins 1-2"

Commit message: hardware: snapshot carrier and face-board integration
Hardware schematics and power:
- complete the BQ25798 charger, TPS61088 5 V boost, MAX17048 gauge, battery controls, and cross-sheet power hierarchy
- add the SN65DSI86 display bridge, HD3SS460 mux, TPS65987D PD controller, USB-C protection, M.2 support, and corrected named-interface wiring
- move the Core2350B0 onto the face-board interconnect, route controls through J25/J2, and make Select directly assert nRPIBOOT
- remove the obsolete J6/J8 expansion headers and move J23 USB-C to the carrier top-left with its VBUS switch and charger support cluster

PCB, footprints, and mechanical assets:
- establish the six-layer controlled-impedance carrier stack, net classes, HDI rules, ground/power planes, keepouts, and placed carrier floorplan
- add the routed two-layer Minerva-Face board with eleven controls, four M2.5 holes, interconnects, fiducials, and a 3.5-inch display datum
- add corrected project-local footprints and STEP models for Core2350B0, USB-C, bridge/PD/power ICs, PicoBlade connectors, M.2 hardware, and critical mechanical envelopes
- correct BAT54 pin mapping, TPS61088 thermal-via numbering, J23 shell geometry, and board-edge lug rules

Verification and reference material:
- add sourcing evidence, ERC/DRC artifacts, STEP assemblies, face render, mechanical coordinates, controlled-impedance notes, and strict connectivity checklists
- document the dock architecture and current board-to-board pin contract
- remove transient root-level DRC and netlist dumps

Torchform and workstation integration:
- fix four-column home navigation and add controller focus/adjustment for quick-settings volume and brightness sliders
- configure Kitty as the terminal backend and add the Minerva SSH workspace folder

Known work-in-progress at this snapshot:
- carrier schematic/PCB parity is clean, but routing remains incomplete at 499 unconnected items with 53 differential-pair tuning violations
- the face board is DRC-clean and f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
Parts:
- removed J8: THD-20-R, Connector_PinSocket_2.54mm:PinSocket_2x20_P2.54mm_Horizontal, symbol Connector_Generic:Conn_02x20_Odd_Even
- BT3: MPN (none) -> ML-1220; Manufacturer (none) -> Panasonic Energy
- C100, C101, C99: MPN (none) -> CC0402KRX5R6BB105; Manufacturer (none) -> Yageo
- C95, C97: MPN (none) -> EMK105B7104KV-F; Manufacturer (none) -> Taiyo Yuden
- C96, C98: MPN (none) -> CL10A106KP8NNNC; Manufacturer (none) -> Samsung Electro-Mechanics
- D1: MPN (none) -> SML-A12U8TT86; Manufacturer (none) -> ROHM
- D2: MPN (none) -> SML-A12M8TT86; Manufacturer (none) -> ROHM
- D6, D7: MPN (none) -> BAT54-7-F; Manufacturer (none) -> Diodes Incorporated
- J14: MPN (none) -> BM04B-SRSS-TB(LF)(SN); Manufacturer (none) -> JST
- J20, J21: MPN (none) -> 53398-0471; Manufacturer (none) -> Molex
- J22: MPN (none) -> BM03B-SRSS-TB(LF)(SN); Manufacturer (none) -> JST
- J25: MPN (none) -> 53047-1410; Manufacturer (none) -> Molex
- Module1: MPN (none) -> CM5008032; Manufacturer (none) -> Raspberry Pi Ltd; Procurement Note (none) -> CM5 8GB LPDDR4X / 32GB eMMC per CONTEXT.md
- R1, R10: MPN (none) -> RK73H1ETTP1001F; Manufacturer (none) -> KOA Speer
- R11: MPN (none) -> RC0402FR-0710KL; Manufacturer (none) -> Yageo
- R4: MPN (none) -> N/A; Manufacturer (none) -> N/A; Procurement Note (none) -> Not fitted
- R5: MPN (none) -> RC0805JR-070RL; Manufacturer (none) -> Yageo
- R71, R72: MPN (none) -> RC0402FR-07100KL; Manufacturer (none) -> Yageo
- R75: MPN (none) -> RC0402FR-071KL; Manufacturer (none) -> Yageo
- R85, R86: MPN (none) -> RT0402FRE072K2L; Manufacturer (none) -> Yageo
- SW1: MPN (none) -> KH-6X6X6H-ZJ; Manufacturer (none) -> Kinghelm; Procurement Note (none) -> Footprint verified against vendor drawing: 4.5 mm signal-pi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
- TP3, TP5: MPN (none) -> N/A; Manufacturer (none) -> PCB fabrication; Procurement Note (none) -> PCB feature; not purchased or placed
- U29: MPN (none) -> PAM8406DR; Manufacturer (none) -> Diodes Incorporated
