File: Minerva-Hardware/CM5_HighSpeed.kicad_sch (KiCad schematic)
At the start: 14 parts, among them J1 HDMI_D_1.4, J16 Conn_01x22_Female, J5 Conn_01x22_Female, J6 THD-02-R, U6 AP22653W6

Commit message: Capture pre-existing Minerva hardware and Torchform work
Hardware schematics and power architecture
- Update carrier, CM5 GPIO, high-speed, PCIe/M.2, face-board, and root schematic hierarchy.
- Add USB-C/DisplayPort dock path, PD controller support, display bridge, audio amplifier, battery charging, boost conversion, fuel gauge, RTC backup, and MCU interconnect changes.
- Add the relocated power/USB schematic and associated local symbols, footprints, and 3D models.

PCB and design assets
- Update the carrier PCB and project configuration.
- Add CM5, connector, power, battery, PD, and board-specific footprint libraries.
- Add the USB-C receptacle STEP model and supporting KiCad assets.
- Apply the surfaced carrier-board geometry cleanup and add the J23 shell-peg DRC rule.

Verification and reference material
- Add CM5 and component datasheets, extracted reference text, current netlist, DRC output, and hardware verification documentation.
- Update CONTEXT.md and workspace metadata with the current project state.

Torchform companion projects
- Add the standalone Qt/QML gamepad prototype.
- Add the Torchform QML GUI shell with screen, panel, radial-menu, keyboard, status, and startup components.
- Add the companion Rust input daemon prototype and configuration.

Project notes
- Add repository guidance and Minerva design/editor notes, including the power-usage note.
Parts:
- removed J16: Conn_01x22_Female, CM5IO:Hirose_FH12-22S-0.5SH_1x22-1MP_P0.50mm_Horizontal, symbol Connector:Conn_01x22_Socket
- removed R8: 2.2K 1%, Resistor_SMD:R_0402_1005Metric, symbol Device:R
- added C70, C71, C72, C73, C74, C80, C81, C88, C89, C91, C92, C93, C94: 100nF, Capacitor_SMD:C_0402_1005Metric, symbol Device:C
- added C75, C76, C82, C83: 10uF, Capacitor_SMD:C_0402_1005Metric, symbol Device:C
- added C77, C78, C79, C84, C85, C90: 1uF, Capacitor_SMD:C_0402_1005Metric, symbol Device:C
- added C86, C87: 390pF, Capacitor_SMD:C_0402_1005Metric, symbol Device:C
- added R50: 51K 1%, Resistor_SMD:R_0402_1005Metric, symbol Device:R
- added R51, R52, R53, R54, R55, R56, R59, R60, R61, R62: 10K, Resistor_SMD:R_0402_1005Metric, symbol Device:R
- added R57, R63, R64, R65, R66: 100K, Resistor_SMD:R_0402_1005Metric, symbol Device:R
- added R58: 1M, Resistor_SMD:R_0402_1005Metric, symbol Device:R
- added U20: SN65DSI86ZQER, Minerva:nFBGA-64_ZQE_5x5mm_P0.5mm, symbol Minerva_Dock:SN65DSI86
- added U21: HD3SS460RHRT, Package_DFN_QFN:WQFN-28-1EP_3.5x5.5mm_P0.5mm_EP2.05x4.05mm_ThermalVias, symbol Minerva_Dock:HD3SS460
- added U22: TPS65987DDJRSHR, Minerva:TPS65987D_VQFN56_RSH, symbol Minerva_Dock:TPS65987D
- added U23: W25Q32JVSS, Package_SO:SOIC-8_5.3x5.3mm_P1.27mm, symbol Memory_Flash:W25Q32JVSS
- added U24: AP2112K-1.8, Package_TO_SOT_SMD:SOT-23-5, symbol Minerva_Dock:LDO_SOT23-5
- added U25: AP2112K-1.2, Package_TO_SOT_SMD:SOT-23-5, symbol Minerva_Dock:LDO_SOT23-5
- J5: footprint CM5IO:Hirose_FH12-22S-0.5SH_1x22-1MP_P0.50mm_Horizontal -> Connector_FFC-FPC:Hirose_FH12-22S-0.5SH_1x22-1MP_P0.50mm_Horizontal
Connections:
- net +3.3v: now also C77.1, C81.1, C82.1, C89.1, C90.1, U21.22 (VCC), U22.5 (VIN_3V3), U24.1 (VIN), U24.3 (EN), U25.1 (VIN), U25.3 (EN)
- net DPHY1_C_N: now also U20.J5 (DACN)
- net DPHY1_C_P: now also U20.H5 (DACP)
- net DPHY1_D0_N: now also U20.J3 (DA0N)
- net DPHY1_D0_P: now also U20.H3 (DA0P)
- net DPHY1_D1_N: now also U20.J4 (DA1N)
- net DPHY1_D1_P: now also U20.H4 (DA1P)
- net DPHY1_D2_N: now also U20.J6 (DA2N)
- net DPHY1_D2_P: now also U20.H6 (DA2P)
- net DPHY1_D3_N: now also U20.J7 (DA3N)
- net DPHY1_D3_P: now also U20.H7 (DA3P)
- net GND: now also C70.2, C71.2, C72.2, C73.2, C74.2, C75.2, C76.2, C77.2, C78.2, C79.2, C80.2, C81.2, C82.2, C83.2, C84.2, C85.2, C86.2, C87.2, C88.2, C89.2, C90.2, R51.2, R52.2, R53.2, R54.2, R55.2, R56.2, R57.2, R58.2, R64.2, R66.2, U20.A1 (ADDR), U20.A7 (REFCLK), U20.A8 (GND), U20.B3 (TEST1), U20.B5 (TEST2), U20.D8 (GND), U20.E4 (GND), U20.E5 (GND), U20.F4 (GND), U20.F5 (GND), U20.F6 (GND), U20.G8 (GND), U21.29 (PAD), U22.1 (PP_HV2), U22.11 (PP_HV1), U22.12 (PP_HV1), U22.2 (PP_HV2), U22.20 (GND), U22.44 (HRESET), U22.45 (GND), U22.46 (GND), U22.47 (GND), U22.51 (GND), U22.59 (PPAD), U23.4 (GND), U24.2 (GND), U25.2 (GND); no longer Module1.157 (USB3-1-RX_N), Module1.159 (USB3-1-RX_P), Module1.163 (USB3-1-D_P), Module1.165 (USB3-1-D_N), Module1.169 (USB3-1-TX_N), Module1.171 (USB3-1-TX_P)
- net SCL1: now also U20.H1 (SCL)
- net SDA1: now also U20.J1 (SDA)
- net VBUS: now also U22.13 (VBUS1), U22.14 (VBUS1), U22.3 (VBUS2), U22.4 (VBUS2)
- new net CC1: C86.1, U22.24 (C_CC1)
- new net CC2: C87.1, U22.26 (C_CC2)
- new net DP_1V2: C70.1, C71.1, C72.1, C75.1, C79.1, U20.A9 (VCCA), U20.B2 (VCCA), U20.D5 (VCC), U20.D6 (VCC), U20.E6 (VCCA), U20.G9 (VCCA), U20.H2 (VCCA), U20.J2 (VCC), U20.J9 (VCC), U25.5 (VOUT)
- new net DP_1V8: C73.1, C74.1, C76.1, C78.1, U20.A2 (VCCIO), U20.B6 (VCCIO), U20.D9 (VPLL), U24.5 (VOUT)
- new net DP_AUX_N: U20.H9 (AUXN), U21.14 (SBU2)
- new net DP_AUX_P: U20.H8 (AUXP), U21.13 (SBU1)
- new net DP_ML0_N: U20.F9 (ML0N), U21.15 (LnAn)
- new net DP_ML0_P: U20.F8 (ML0P), U21.16 (LnAp)
- new net DP_ML1_N: U20.E9 (ML1N), U21.18 (LnBn)
- new net DP_ML1_P: U20.E8 (ML1P), U21.19 (LnBp)
- new net DSI86_EN: R55.1, U20.B1 (EN)
- new net DSI86_HPD: R50.1, U20.J8 (HPD)
- new net DSI86_IRQ: U20.A3 (IRQ)
- new net DSI86_STRAP1: R51.1, U20.A4 (GPIO1)
- new net DSI86_STRAP2: R52.1, U20.A5 (GPIO2)
- new net DSI86_STRAP3: R53.1, U20.A6 (GPIO3)
- new net DSI86_STRAP4: R54.1, U20.B4 (GPIO4)
- new net DSI86_TEST3: C80.1, U20.B7 (TEST3)
- new net HD_TX1_N: C92.1, U21.5 (CTX1n)
- new net HD_TX1_P: C91.1, U21.4 (CTX1p)
- new net HD_TX2_N: C94.1, U21.7 (CTX2n)
- new net HD_TX2_P: C93.1, U21.6 (CTX2p)
- new net MUX_AMSEL: R56.1, U21.8 (AMSEL)
- new net MUX_EN: R57.1, U21.17 (EN), U22.31 (GPIO4)
- new net MUX_POL: U21.3 (POL), U22.18 (GPIO2)
- new net PD_HPD_SRC: R50.2, U22.30 (GPIO3_HPD)
- new net PD_I2C_IRQ: R62.2, U22.29 (I2C1_IRQ)
- new net PD_I2C_SCL: R60.2, U22.27 (I2C1_SCL)
- new net PD_I2C_SDA: R61.2, U22.28 (I2C1_SDA)
- new net TPS_ADCIN1: R63.2, R64.1, U22.6 (ADCIN1)
- new net TPS_ADCIN2: R65.2, R66.1, U22.10 (ADCIN2)
- new net TPS_DRAIN1: U22.15 (DRAIN1), U22.19 (DRAIN1), U22.58 (DRAIN1), U22.8 (DRAIN1)
- new net TPS_DRAIN2: U22.52 (DRAIN2), U22.56 (DRAIN2), U22.57 (DRAIN2), U22.7 (DRAIN2)
- new net TPS_GPIO0: U22.16 (GPIO0)
- new net TPS_GPIO1: R58.1, U22.17 (GPIO1)
- new net TPS_LDO_1V8: C84.1, U22.35 (LDO_1V8)
- new net TPS_LDO_3V3: C83.1, C88.1, R59.1, R60.1, R61.1, R62.1, R63.1, R65.1, U22.9 (LDO_3V3), U23.3 (~{WP}/IO_{2}), U23.7 (~{HOLD}/~{RESET}/IO_{3}), U23.8 (VCC)
- new net TPS_PP_CABLE: C85.1, U22.25 (PP_CABLE)
- new net TPS_SPI_CLK: U22.38 (SPI_CLK), U23.6 (CLK)
- new net TPS_SPI_CS: R59.2, U22.39 (SPI_CS), U23.1 (~{CS})
- new net TPS_SPI_PICO: U22.37 (SPI_PICO), U23.5 (DI/IO_{0})
- new net TPS_SPI_POCI: U22.36 (SPI_POCI), U23.2 (DO/IO_{1})
- new net USB3-1-D_N: Module1.165 (USB3-1-D_N)
- new net USB3-1-D_P: Module1.163 (USB3-1-D_P)
- new net USB3-1-RX_N: Module1.157 (USB3-1-RX_N), U21.27 (SSRXn)
- new net USB3-1-RX_P: Module1.159 (USB3-1-RX_P), U21.28 (SSRXp)
- new net USB3-1-TX_N: Module1.169 (USB3-1-TX_N), U21.25 (SSTXn)
- new net USB3-1-TX_P: Module1.171 (USB3-1-TX_P), U21.26 (SSTXp)
- new net USBC_RX1_N: U21.2 (CRX1n)
- new net USBC_RX1_P: U21.1 (CRX1p)
- new net USBC_RX2_N: U21.10 (CRX2n)
- new net USBC_RX2_P: U21.9 (CRX2p)
- new net USBC_SBU1: U21.11 (CSBU1)
- new net USBC_SBU2: U21.12 (CSBU2)
- new net USBC_TX1_N: C92.2
- new net USBC_TX1_P: C91.2
- new net USBC_TX2_N: C94.2
- new net USBC_TX2_P: C93.2
- no-connect marks 21 -> 52
Other:
- note added: "Global labels: USBC_* SS/SBU pairs to J23 receptacle on root sheet."
- note added: "USB-C DOCK CHAIN (DP alt mode) U20 SN65DSI86: DSI1 (DPHY1) -> 2-lane DP HBR2. REFCLK=GND: DP PLL fed from DSI clock (mainline ti-sn65dsi86 driver, I2C addr 0x2C on SDA1/SCL1). ML2/ML3 unused. U21 HD3SS460 assignment-D combo: ML0->LnA, ML1->LnB, LnC/LnD open (Table 3, SLLSEM7D). USBC_TX/RX/SBU nets -> 24-pin USB-C receptacle SS pins (receptacle TBD). U22 TPS65987D: DRP, power sink / DP source. CC1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"
- note added: "Upper display: HDMI0 over FFC ribbon = J1 (HDMI_D_1.4). DSI1 is dedicated to U20 SN65DSI86 (USB-C DP out). Lower display: J5 = DSI0 + I2C0 touch (SPI alternative available on 40-pin header J8)."

Commit message: hardware: snapshot carrier and face-board integration
Hardware schematics and power:
- complete the BQ25798 charger, TPS61088 5 V boost, MAX17048 gauge, battery controls, and cross-sheet power hierarchy
- add the SN65DSI86 display bridge, HD3SS460 mux, TPS65987D PD controller, USB-C protection, M.2 support, and corrected named-interface wiring
- move the Core2350B0 onto the face-board interconnect, route controls through J25/J2, and make Select directly assert nRPIBOOT
- remove the obsolete J6/J8 expansion headers and move J23 USB-C to the carrier top-left with its VBUS switch and charger support cluster

PCB, footprints, and mechanical assets:
- establish the six-layer controlled-impedance carrier stack, net classes, HDI rules, ground/power planes, keepouts, and placed carrier floorplan
- add the routed two-layer Minerva-Face board with eleven controls, four M2.5 holes, interconnects, fiducials, and a 3.5-inch display datum
- add corrected project-local footprints and STEP models for Core2350B0, USB-C, bridge/PD/power ICs, PicoBlade connectors, M.2 hardware, and critical mechanical envelopes
- correct BAT54 pin mapping, TPS61088 thermal-via numbering, J23 shell geometry, and board-edge lug rules

Verification and reference material:
- add sourcing evidence, ERC/DRC artifacts, STEP assemblies, face render, mechanical coordinates, controlled-impedance notes, and strict connectivity checklists
- document the dock architecture and current board-to-board pin contract
- remove transient root-level DRC and netlist dumps

Torchform and workstation integration:
- fix four-column home navigation and add controller focus/adjustment for quick-settings volume and brightness sliders
- configure Kitty as the terminal backend and add the Minerva SSH workspace folder

Known work-in-progress at this snapshot:
- carrier schematic/PCB parity is clean, but routing remains incomplete at 499 unconnected items with 53 differential-pair tuning violations
- the face board is DRC-clean and f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
Parts:
- removed J6: THD-02-R, Connector_PinHeader_2.54mm:PinHeader_2x02_P2.54mm_Vertical, symbol Connector_Generic:Conn_02x02_Odd_Even
- C2, C7, C8: MPN (none) -> CL21A106KPFNNNE; Manufacturer (none) -> Samsung Electro-Mechanics
- C3: MPN (none) -> T491D107K010AT; Manufacturer (none) -> KEMET
- C70, C71, C72, C73, C74, C80, C81, C88, C89, C91, C92, C93, C94: MPN (none) -> EMK105B7104KV-F; Manufacturer (none) -> Taiyo Yuden
- C75, C76, C82, C83: footprint Capacitor_SMD:C_0402_1005Metric -> Capacitor_SMD:C_0603_1608Metric; MPN (none) -> CL10A106KP8NNNC; Manufacturer (none) -> Samsung Electro-Mechanics
- C77, C78, C79, C84, C85, C90: MPN (none) -> CC0402KRX5R6BB105; Manufacturer (none) -> Yageo
- C86, C87: MPN (none) -> GRM1555C1H391JA01D; Manufacturer (none) -> Murata
- J1: MPN (none) -> 2-1734839-0; Manufacturer (none) -> TE Connectivity
- J5: MPN (none) -> FH12-22S-0.5SH(55); Manufacturer (none) -> Hirose
- Module1: MPN (none) -> CM5008032; Manufacturer (none) -> Raspberry Pi Ltd; Procurement Note (none) -> CM5 8GB LPDDR4X / 32GB eMMC per CONTEXT.md
- R12: MPN (none) -> CRCW040215K0FKED; Manufacturer (none) -> Vishay
- R50: MPN (none) -> RC0402FR-0751KL; Manufacturer (none) -> Yageo
- R51, R52, R53, R54, R55, R56, R59, R60, R61, R62: MPN (none) -> RC0402FR-0710KL; Manufacturer (none) -> Yageo
- R57, R63, R64, R65, R66: MPN (none) -> RC0402FR-07100KL; Manufacturer (none) -> Yageo
- R58: MPN (none) -> RC0402FR-071ML; Manufacturer (none) -> Yageo
- R6, R7: MPN (none) -> RT0402FRE072K2L; Manufacturer (none) -> Yageo
- U20: MPN (none) -> SN65DSI86ZQER; Manufacturer (none) -> Texas Instruments
- U21: MPN (none) -> HD3SS460RHRT; Manufacturer (none) -> Texas Instruments
- U22: MPN (none) -> TPS65987DDJRSHR; Manufacturer (none) -> Texas Instruments
- U23: MPN (none) -> W25Q32JVSSIQ; Manufacturer (none) -> Winbond
- U24: MPN (none) -> AP2112K-1.8TRG1; Manufacturer (none) -> Diodes Incorporated
- U25: MPN (none) -> AP2112K-1.2TRG1; Manufacturer (none) -> Diodes Incorporated
- U6: MPN (none) -> AP22653W6-7; Manufacturer (none) -> Diodes Incorporated
Other:
- note added: "Debug: ID_SC/ID_SD on J8 pins 27/28; DSI86 I2C (SDA1/SCL1) probe at R6/R7. (J6 header removed - no board space.)"
