File: Minerva-Hardware/face_board.kicad_sch (KiCad schematic)
At the start: 12 parts, among them SW10 SW_Push, SW11 SW_Push, SW12 SW_Push, SW2 SW_Push, SW3 SW_Push, SW4 SW_Push, SW5 SW_Push, SW6 SW_Push, SW7 SW_Push, SW8 SW_Push, SW9 SW_Push

Commit message: Capture pre-existing Minerva hardware and Torchform work
Hardware schematics and power architecture
- Update carrier, CM5 GPIO, high-speed, PCIe/M.2, face-board, and root schematic hierarchy.
- Add USB-C/DisplayPort dock path, PD controller support, display bridge, audio amplifier, battery charging, boost conversion, fuel gauge, RTC backup, and MCU interconnect changes.
- Add the relocated power/USB schematic and associated local symbols, footprints, and 3D models.

PCB and design assets
- Update the carrier PCB and project configuration.
- Add CM5, connector, power, battery, PD, and board-specific footprint libraries.
- Add the USB-C receptacle STEP model and supporting KiCad assets.
- Apply the surfaced carrier-board geometry cleanup and add the J23 shell-peg DRC rule.

Verification and reference material
- Add CM5 and component datasheets, extracted reference text, current netlist, DRC output, and hardware verification documentation.
- Update CONTEXT.md and workspace metadata with the current project state.

Torchform companion projects
- Add the standalone Qt/QML gamepad prototype.
- Add the Torchform QML GUI shell with screen, panel, radial-menu, keyboard, status, and startup components.
- Add the companion Rust input daemon prototype and configuration.

Project notes
- Add repository guidance and Minerva design/editor notes, including the power-usage note.
Parts:
- removed A1: RaspberryPi_Pico, Module:RaspberryPi_Pico_Common_Unspecified, symbol MCU_Module:RaspberryPi_Pico
- added A1: Core2350B, Minerva:Core2350B_stamp64, symbol Minerva_Dock:Core2350B
- added J2: CARRIER 14P, Connector_Molex:Molex_PicoBlade_53047-1410_1x14_P1.25mm_Vertical, symbol Connector_Generic:Conn_01x14
- added J3: SHOULDER 6P, Connector_Molex:Molex_PicoBlade_53047-0610_1x06_P1.25mm_Vertical, symbol Connector_Generic:Conn_01x06
- SW10, SW11, SW12, SW2, SW3, SW4, SW5, SW6, SW7, SW8, SW9: footprint (none) -> Button_Switch_SMD:SW_SPST_SKQG_WithStem
Connections:
- net +5V: now also A1.31 (VBUS), J2.1 (Pin_1)
- net BUT_A: now also A1.13 (GP12)
- net BUT_B: now also A1.16 (GP13)
- net BUT_DOWN: now also A1.38 (GP18)
- net BUT_HOME: now also A1.46 (GP26)
- net BUT_L: now also A1.40 (GP20), J3.1 (Pin_1)
- net BUT_LEFT: now also A1.37 (GP19)
- net BUT_R: now also A1.42 (GP22), J3.4 (Pin_4)
- net BUT_RIGHT: now also A1.35 (GP17)
- net BUT_SEL: now also A1.43 (GP25)
- net BUT_START: now also A1.44 (GP24)
- net BUT_UP: now also A1.36 (GP16)
- net BUT_X: now also A1.15 (GP14)
- net BUT_Y: now also A1.34 (GP15)
- net BUT_ZL: now also A1.39 (GP21), J3.2 (Pin_2)
- net BUT_ZR: now also A1.41 (GP23), J3.5 (Pin_5)
- net GND: now also A1.1 (GND), A1.17 (GND), A1.24 (GND), A1.30 (GND), A1.33 (GND), A1.49 (GND), J2.14 (Pin_14), J2.2 (Pin_2), J3.3 (Pin_3), J3.6 (Pin_6)
- new net AMP_nMUTE: A1.9 (GP8), J2.12 (Pin_12)
- new net AMP_nSD: A1.12 (GP9), J2.13 (Pin_13)
- new net BQ_SCL: A1.10 (GP7), J2.9 (Pin_9)
- new net BQ_SDA: A1.7 (GP6), J2.8 (Pin_8)
- new net PD_I2C_IRQ: A1.3 (GP2), J2.5 (Pin_5)
- new net PD_I2C_SCL: A1.4 (GP1), J2.4 (Pin_4)
- new net PD_I2C_SDA: A1.2 (GP0), J2.3 (Pin_3)
- new net PWR_BUT: A1.11 (GP10), J2.10 (Pin_10)
- new net RP_3V3: A1.32 (3V3)
- new net RP_BOOTSEL: A1.21 (BOOTSEL)
- new net RP_RUN: A1.27 (RUN)
- new net RP_SWCLK: A1.26 (SWCLK)
- new net RP_SWDIO: A1.22 (SWDIO)
- new net RP_USB_N: A1.23 (USBD_N)
- new net RP_USB_P: A1.25 (USBD_P)
- new net SCL_I2C: A1.8 (GP5), J2.7 (Pin_7)
- new net SDA_I2C: A1.5 (GP4), J2.6 (Pin_6)
- new net nRPIBOOT: A1.14 (GP11), J2.11 (Pin_11)
- no-connect marks 1 -> 24
Other:
- note added: "RP2350B debug: RP_SWDIO/RP_SWCLK/RP_USB_* stubs - fit header if needed"
- note added: "Rails fed from carrier via J2"

Commit message: hardware: snapshot carrier and face-board integration
Hardware schematics and power:
- complete the BQ25798 charger, TPS61088 5 V boost, MAX17048 gauge, battery controls, and cross-sheet power hierarchy
- add the SN65DSI86 display bridge, HD3SS460 mux, TPS65987D PD controller, USB-C protection, M.2 support, and corrected named-interface wiring
- move the Core2350B0 onto the face-board interconnect, route controls through J25/J2, and make Select directly assert nRPIBOOT
- remove the obsolete J6/J8 expansion headers and move J23 USB-C to the carrier top-left with its VBUS switch and charger support cluster

PCB, footprints, and mechanical assets:
- establish the six-layer controlled-impedance carrier stack, net classes, HDI rules, ground/power planes, keepouts, and placed carrier floorplan
- add the routed two-layer Minerva-Face board with eleven controls, four M2.5 holes, interconnects, fiducials, and a 3.5-inch display datum
- add corrected project-local footprints and STEP models for Core2350B0, USB-C, bridge/PD/power ICs, PicoBlade connectors, M.2 hardware, and critical mechanical envelopes
- correct BAT54 pin mapping, TPS61088 thermal-via numbering, J23 shell geometry, and board-edge lug rules

Verification and reference material:
- add sourcing evidence, ERC/DRC artifacts, STEP assemblies, face render, mechanical coordinates, controlled-impedance notes, and strict connectivity checklists
- document the dock architecture and current board-to-board pin contract
- remove transient root-level DRC and netlist dumps

Torchform and workstation integration:
- fix four-column home navigation and add controller focus/adjustment for quick-settings volume and brightness sliders
- configure Kitty as the terminal backend and add the Minerva SSH workspace folder

Known work-in-progress at this snapshot:
- carrier schematic/PCB parity is clean, but routing remains incomplete at 499 unconnected items with 53 differential-pair tuning violations
- the face board is DRC-clean and f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
Parts:
- A1: value Core2350B -> Core2350B0; MPN (none) -> Core2350B0; Manufacturer (none) -> Waveshare; Procurement Note (none) -> 0 MB PSRAM variant selected; 16 MB flash and 520 KB interna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
- J2: MPN (none) -> 53047-1410; Manufacturer (none) -> Molex; Procurement Note (none) -> PicoBlade 1.25 mm, vertical through-hole, 14 circuits.
- J3: MPN (none) -> 53047-0610; Manufacturer (none) -> Molex; Procurement Note (none) -> PicoBlade 1.25 mm, vertical through-hole, 6 circuits.
- SW10, SW11, SW12, SW2, SW3, SW4, SW5, SW6, SW7, SW8, SW9: value SW_Push -> SKQGAFE010; MPN (none) -> SKQGAFE010; Manufacturer (none) -> Alps Alpine
Connections:
- net BUT_SEL is gone; now on net nRPIBOOT: A1.43 (GP25), SW11.1
- net nRPIBOOT: no longer A1.14 (GP11)
- no-connect marks 24 -> 25
